Commit message: Convert non-standard material_name to standard <material> element and format XML
- Replace material_name="xxx" attribute on <mesh> with <material name="xxx"/>
  child element under <visual> (73 visual blocks in 15 files)
- Format all .urdf/.robot/.positioner/.track files with consistent 2-space
  indentation, preserving XML declarations, comments, and all content values

Co-Authored-By: Claude Opus 4.6 <noreply@anthropic.com>

File: Robots/COMAU_ComauSMART_NJ_500-2.7/COMAU_ComauSMART_NJ_500-2.7.urdf (robot description, URDF)
Before this commit: robot COMAU_ComauSMART_NJ_500-2.7, 8 links, 7 joints
Links:
- link base_link: geometry collision mesh filename=collision/base_link.stl; visual mesh filename=visual/base_link.stl
- link link1: geometry collision mesh filename=collision/link1.stl; visual mesh filename=visual/link_1.stl
- link link2: geometry collision mesh filename=collision/link2.stl; visual mesh filename=visual/link_2.stl
- link link3: geometry collision mesh filename=collision/link3.stl; visual mesh filename=visual/link_3.stl
- link link4: geometry collision mesh filename=collision/link4.stl; visual mesh filename=visual/link_4.stl
- link link5: geometry collision mesh filename=collision/link5.stl; visual mesh filename=visual/link_5.stl
- link link6: geometry collision mesh filename=collision/link6.stl; visual mesh filename=visual/link_6.stl

File: Robots/CUSTOM_Gantry/CUSTOM_Gantry.urdf (robot description, URDF)
Before this commit: robot CUSTOM_Gantry, 8 links, 7 joints
Links:
- link base_link: geometry collision mesh filename=collision/base_link.stl; visual mesh filename=visual/base_link.stl
- link link2: geometry collision mesh filename=collision/link2.stl; visual mesh filename=visual/link_2.stl
- link link3: geometry collision mesh filename=collision/link3.stl; visual mesh filename=visual/link_3.stl
- link link4: geometry collision mesh filename=collision/link4.stl; visual mesh filename=visual/link_4.stl
- link link5: geometry collision mesh filename=collision/link5.stl; visual mesh filename=visual/link_5.stl
- link link6: geometry collision mesh filename=collision/link6.stl; visual mesh filename=visual/link_6.stl
- link link_1: geometry collision mesh filename=collision/link_1.stl; visual mesh filename=visual/link_1.stl

File: Robots/CUSTOM_TapePlacementGantry/CUSTOM_TapePlacementGantry.urdf (robot description, URDF)
Before this commit: robot CUSTOM_TapePlacementGantry, 6 links, 5 joints
Links:
- link base_link: geometry collision mesh filename=collision/base_link.stl; visual mesh filename=visual/base_link.stl
- link link1: geometry collision mesh filename=collision/link1.stl; visual mesh filename=visual/link_1.stl
- link link2: geometry collision mesh filename=collision/link2.stl; visual mesh filename=visual/link_2.stl
- link link3: geometry collision mesh filename=collision/link3.stl; visual mesh filename=visual/link_3.stl
- link link4: geometry collision mesh filename=collision/link4.stl; visual mesh filename=visual/link_4.stl

File: Robots/INOVANCE_IR-R35JQR/INOVANCE_IR-R35JQR.urdf (robot description, URDF)
Before this commit: robot INOVANCE_IR-R35JQR, 8 links, 7 joints
Links:
- link base_link: geometry collision mesh filename=collision/base_link.stl; visual mesh filename=visual/base_link.stl
- link link1: geometry collision mesh filename=collision/link1.stl; visual mesh filename=visual/link_1.stl
- link link2: geometry collision mesh filename=collision/link2.stl; visual mesh filename=visual/link_2.stl
- link link3: geometry collision mesh filename=collision/link3.stl; visual mesh filename=visual/link_3.stl
- link link4: geometry collision mesh filename=collision/link4.stl; visual mesh filename=visual/link_4.stl
- link link5: geometry collision mesh filename=collision/link5.stl; visual mesh filename=visual/link_5.stl
- link link6: geometry collision mesh filename=collision/link6.stl; visual mesh filename=visual/link_6.stl

File: Robots/KUKA_KR10R1420HP/KUKA_KR10R1420HP.urdf (robot description, URDF)
Before this commit: robot KUKA_KR10R1420HP, 8 links, 7 joints
Links:
- link base_link: geometry collision mesh filename=collision/base_link.stl; visual mesh filename=visual/base_link.stl
- link link1: geometry collision mesh filename=collision/link1.stl; visual mesh filename=visual/link_1.stl
- link link2: geometry collision mesh filename=collision/link2.stl; visual mesh filename=visual/link_2.stl
- link link3: geometry collision mesh filename=collision/link3.stl; visual mesh filename=visual/link_3.stl
- link link4: geometry collision mesh filename=collision/link4.stl; visual mesh filename=visual/link_4.stl
- link link5: geometry collision mesh filename=collision/link5.stl; visual mesh filename=visual/link_5.stl
- link link6: geometry collision mesh filename=collision/link6.stl; visual mesh filename=visual/link_6.stl

File: Robots/KUKA_KR210R2700-2/KUKA_KR210R2700-2.urdf (robot description, URDF)
Before this commit: robot KUKA_KR210R2700-2, 8 links, 7 joints
Links:
- link base_link: geometry collision mesh filename=collision/base_link.stl; visual mesh filename=visual/base_link.stl
- link link1: geometry collision mesh filename=collision/link1.stl; visual mesh filename=visual/link_1.stl
- link link2: geometry collision mesh filename=collision/link2.stl; visual mesh filename=visual/link_2.stl
- link link3: geometry collision mesh filename=collision/link3.stl; visual mesh filename=visual/link_3.stl
- link link4: geometry collision mesh filename=collision/link4.stl; visual mesh filename=visual/link_4.stl
- link link5: geometry collision mesh filename=collision/link5.stl; visual mesh filename=visual/link_5.stl
- link link6: geometry collision mesh filename=collision/link6.stl; visual mesh filename=visual/link_6.stl

File: Robots/KUKA_KR360R2830/KUKA_KR360R2830.urdf (robot description, URDF)
Before this commit: robot KUKA_KR360R2830, 8 links, 7 joints
Links:
- link base_link: geometry collision mesh filename=collision/base_link.stl; visual mesh filename=visual/base_link.stl
- link link1: geometry collision mesh filename=collision/link1.stl; visual mesh filename=visual/link_1.stl
- link link2: geometry collision mesh filename=collision/link2.stl; visual mesh filename=visual/link_2.stl
- link link3: geometry collision mesh filename=collision/link3.stl; visual mesh filename=visual/link_3.stl
- link link4: geometry collision mesh filename=collision/link4.stl; visual mesh filename=visual/link_4.stl
- link link5: geometry collision mesh filename=collision/link5.stl; visual mesh filename=visual/link_5.stl
- link link6: geometry collision mesh filename=collision/link6.stl; visual mesh filename=visual/link_6.stl

File: Robots/KUKA_KR480R3330MT/KUKA_KR480R3330MT.urdf (robot description, URDF)
Before this commit: robot KUKA_KR480R3330MT, 8 links, 7 joints
Links:
- link base_link: geometry collision mesh filename=collision/base_link.stl; visual mesh filename=visual/base_link.stl
- link link1: geometry collision mesh filename=collision/link1.stl; visual mesh filename=visual/link_1.stl
- link link2: geometry collision mesh filename=collision/link2.stl; visual mesh filename=visual/link_2.stl
- link link3: geometry collision mesh filename=collision/link3.stl; visual mesh filename=visual/link_3.stl
- link link4: geometry collision mesh filename=collision/link4.stl; visual mesh filename=visual/link_4.stl
- link link5: geometry collision mesh filename=collision/link5.stl; visual mesh filename=visual/link_5.stl
- link link6: geometry collision mesh filename=collision/link6.stl; visual mesh filename=visual/link_6.stl

File: Robots/KUKA_KR500R2380/KUKA_KR500R2380.urdf (robot description, URDF)
Before this commit: robot KUKA_KR500R2380, 8 links, 7 joints
Links:
- link base_link: geometry collision mesh filename=collision/base_link.stl; visual mesh filename=visual/base_link.stl
- link link1: geometry collision mesh filename=collision/link1.stl; visual mesh filename=visual/link_1.stl
- link link2: geometry collision mesh filename=collision/link2.stl; visual mesh filename=visual/link_2.stl
- link link3: geometry collision mesh filename=collision/link3.stl; visual mesh filename=visual/link_3.stl
- link link4: geometry collision mesh filename=collision/link4.stl; visual mesh filename=visual/link_4.stl
- link link5: geometry collision mesh filename=collision/link5.stl; visual mesh filename=visual/link_5.stl
- link link6: geometry collision mesh filename=collision/link6.stl; visual mesh filename=visual/link_6.stl
