Commit message: add missing collision meshes

File: Robots/COMAU_ComauSMART_NJ_500-2.7/COMAU_ComauSMART_NJ_500-2.7.urdf (robot description, URDF)
Before this commit: robot COMAU_ComauSMART_NJ_500-2.7, 8 links, 7 joints
Links:
- link base_link: geometry collision mesh filename=collision/base_link.stl; visual mesh filename=visual/base_link.stl material_name=gray
- link link1: geometry collision mesh filename=collision/link1.stl; visual mesh filename=visual/link_1.stl material_name=comau_red
- link link2: geometry collision mesh filename=collision/link2.stl; visual mesh filename=visual/link_2.stl material_name=comau_red
- link link3: geometry collision mesh filename=collision/link3.stl; visual mesh filename=visual/link_3.stl material_name=comau_red
- link link4: geometry collision mesh filename=collision/link4.stl; visual mesh filename=visual/link_4.stl material_name=comau_red
- link link5: geometry collision mesh filename=collision/link5.stl; visual mesh filename=visual/link_5.stl material_name=comau_red
- link link6: geometry collision mesh filename=collision/link6.stl; visual mesh filename=visual/link_6.stl material_name=comau_red

File: Robots/CUSTOM_Gantry/CUSTOM_Gantry.urdf (robot description, URDF)
Before this commit: robot CUSTOM_Gantry, 8 links, 7 joints
Links:
- link base_link: geometry collision mesh filename=collision/base_link.stl; visual mesh filename=visual/base_link.stl material_name=gantry_gray
- link link2: geometry collision mesh filename=collision/link2.stl; visual mesh filename=visual/link_2.stl material_name=gantry_white
- link link3: geometry collision mesh filename=collision/link3.stl; visual mesh filename=visual/link_3.stl material_name=gantry_white
- link link4: geometry collision mesh filename=collision/link4.stl; visual mesh filename=visual/link_4.stl material_name=gantry_white
- link link5: geometry collision mesh filename=collision/link5.stl; visual mesh filename=visual/link_5.stl material_name=gantry_white
- link link6: geometry collision mesh filename=collision/link6.stl; visual mesh filename=visual/link_6.stl material_name=gantry_white
- link link_1: geometry collision mesh filename=collision/link_1.stl; visual mesh filename=visual/link_1.stl material_name=gantry_white

File: Robots/CUSTOM_TapePlacementGantry/CUSTOM_TapePlacementGantry.urdf (robot description, URDF)
Before this commit: robot CUSTOM_TapePlacementGantry, 6 links, 5 joints
Links:
- link base_link: geometry collision mesh filename=collision/base_link.stl; visual mesh filename=visual/base_link.stl material_name=gantry_gray
- link link1: geometry collision mesh filename=collision/link1.stl; visual mesh filename=visual/link_1.stl material_name=gantry_organge
- link link2: geometry collision mesh filename=collision/link2.stl; visual mesh filename=visual/link_2.stl material_name=gantry_lightgreen
- link link3: geometry collision mesh filename=collision/link3.stl; visual mesh filename=visual/link_3.stl material_name=gantry_purple
- link link4: geometry collision mesh filename=collision/link4.stl; visual mesh filename=visual/link_4.stl material_name=gantry_deepblue

File: Robots/INOVANCE_IR-R35JQR/INOVANCE_IR-R35JQR.urdf (robot description, URDF)
Before this commit: robot INOVANCE_IR-R35JQR, 8 links, 7 joints
Links:
- link base_link: geometry collision mesh filename=collision/base_link.stl; visual mesh filename=visual/base_link.stl material_name=kuka_gray
- link link1: geometry collision mesh filename=collision/link1.stl; visual mesh filename=visual/link_1.stl material_name=kuka_organge
- link link2: geometry collision mesh filename=collision/link2.stl; visual mesh filename=visual/link_2.stl material_name=kuka_organge
- link link3: geometry collision mesh filename=collision/link3.stl; visual mesh filename=visual/link_3.stl material_name=kuka_organge
- link link4: geometry collision mesh filename=collision/link4.stl; visual mesh filename=visual/link_4.stl material_name=kuka_organge
- link link5: geometry collision mesh filename=collision/link5.stl; visual mesh filename=visual/link_5.stl material_name=kuka_organge
- link link6: geometry collision mesh filename=collision/link6.stl; visual mesh filename=visual/link_6.stl material_name=kuka_organge

File: Robots/KUKA_KR10R1420HP/KUKA_KR10R1420HP.urdf (robot description, URDF)
Before this commit: robot KUKA_KR10R1420HP, 8 links, 7 joints
Links:
- link base_link: geometry collision mesh filename=collision/base_link.stl; visual mesh filename=visual/base_link.stl material_name=kuka_gray
- link link1: geometry collision mesh filename=collision/link1.stl; visual mesh filename=visual/link_1.stl material_name=kuka_organge
- link link2: geometry collision mesh filename=collision/link2.stl; visual mesh filename=visual/link_2.stl material_name=kuka_organge
- link link3: geometry collision mesh filename=collision/link3.stl; visual mesh filename=visual/link_3.stl material_name=kuka_organge
- link link4: geometry collision mesh filename=collision/link4.stl; visual mesh filename=visual/link_4.stl material_name=kuka_organge
- link link5: geometry collision mesh filename=collision/link5.stl; visual mesh filename=visual/link_5.stl material_name=kuka_organge
- link link6: geometry collision mesh filename=collision/link6.stl; visual mesh filename=visual/link_6.stl material_name=kuka_organge

File: Robots/KUKA_KR210R2700-2/KUKA_KR210R2700-2.urdf (robot description, URDF)
Before this commit: robot KUKA_KR210R2700-2, 8 links, 7 joints
Links:
- link base_link: geometry collision mesh filename=collision/base_link.stl; visual mesh filename=visual/base_link.stl material_name=kuka_gray
- link link1: geometry collision mesh filename=collision/link1.stl; visual mesh filename=visual/link_1.stl material_name=kuka_organge
- link link2: geometry collision mesh filename=collision/link2.stl; visual mesh filename=visual/link_2.stl material_name=kuka_organge
- link link3: geometry collision mesh filename=collision/link3.stl; visual mesh filename=visual/link_3.stl material_name=kuka_organge
- link link4: geometry collision mesh filename=collision/link4.stl; visual mesh filename=visual/link_4.stl material_name=kuka_organge
- link link5: geometry collision mesh filename=collision/link5.stl; visual mesh filename=visual/link_5.stl material_name=kuka_organge
- link link6: geometry collision mesh filename=collision/link6.stl; visual mesh filename=visual/link_6.stl material_name=kuka_organge

File: Robots/KUKA_KR360R2830/KUKA_KR360R2830.urdf (robot description, URDF)
Before this commit: robot KUKA_KR360R2830, 8 links, 7 joints
Links:
- link base_link: geometry collision mesh filename=collision/base_link.stl; visual mesh filename=visual/base_link.stl material_name=kuka_gray
- link link1: geometry collision mesh filename=collision/link1.stl; visual mesh filename=visual/link_1.stl material_name=kuka_organge
- link link2: geometry collision mesh filename=collision/link2.stl; visual mesh filename=visual/link_2.stl material_name=kuka_organge
- link link3: geometry collision mesh filename=collision/link3.stl; visual mesh filename=visual/link_3.stl material_name=kuka_organge
- link link4: geometry collision mesh filename=collision/link4.stl; visual mesh filename=visual/link_4.stl material_name=kuka_organge
- link link5: geometry collision mesh filename=collision/link5.stl; visual mesh filename=visual/link_5.stl material_name=kuka_organge
- link link6: geometry collision mesh filename=collision/link6.stl; visual mesh filename=visual/link_6.stl material_name=kuka_organge

File: Robots/KUKA_KR480R3330MT/KUKA_KR480R3330MT.urdf (robot description, URDF)
Before this commit: robot KUKA_KR480R3330MT, 8 links, 7 joints
Links:
- link base_link: geometry collision mesh filename=collision/base_link.stl; visual mesh filename=visual/base_link.stl material_name=kuka_gray
- link link1: geometry collision mesh filename=collision/link1.stl; visual mesh filename=visual/link_1.stl material_name=kuka_organge
- link link2: geometry collision mesh filename=collision/link2.stl; visual mesh filename=visual/link_2.stl material_name=kuka_organge
- link link3: geometry collision mesh filename=collision/link3.stl; visual mesh filename=visual/link_3.stl material_name=kuka_organge
- link link4: geometry collision mesh filename=collision/link4.stl; visual mesh filename=visual/link_4.stl material_name=kuka_organge
- link link5: geometry collision mesh filename=collision/link5.stl; visual mesh filename=visual/link_5.stl material_name=kuka_organge
- link link6: geometry collision mesh filename=collision/link6.stl; visual mesh filename=visual/link_6.stl material_name=kuka_organge

File: Robots/KUKA_KR500R2380/KUKA_KR500R2380.urdf (robot description, URDF)
Before this commit: robot KUKA_KR500R2380, 8 links, 7 joints
Links:
- link base_link: geometry collision mesh filename=collision/base_link.stl; visual mesh filename=visual/base_link.stl material_name=kuka_gray
- link link1: geometry collision mesh filename=collision/link1.stl; visual mesh filename=visual/link_1.stl material_name=kuka_organge
- link link2: geometry collision mesh filename=collision/link2.stl; visual mesh filename=visual/link_2.stl material_name=kuka_organge
- link link3: geometry collision mesh filename=collision/link3.stl; visual mesh filename=visual/link_3.stl material_name=kuka_organge
- link link4: geometry collision mesh filename=collision/link4.stl; visual mesh filename=visual/link_4.stl material_name=kuka_organge
- link link5: geometry collision mesh filename=collision/link5.stl; visual mesh filename=visual/link_5.stl material_name=kuka_organge
- link link6: geometry collision mesh filename=collision/link6.stl; visual mesh filename=visual/link_6.stl material_name=kuka_organge

File: Robots/MOTOMAN_GP225/MOTOMAN_GP225.urdf (robot description, URDF)
Before this commit: robot MOTOMAN_GP225, 12 links, 11 joints
Links:
- link link_2_l_2: geometry collision mesh filename=collision/link_2_l_2.stl; visual mesh filename=visual/link_2_l_2.dae

Commit message: Update upload_to_r2.py to support update-file filtering, and update COMAU and CUSTOM gantries URDFs

File: Robots/COMAU_ComauSMART_NJ_500-2.7/COMAU_ComauSMART_NJ_500-2.7.urdf (robot description, URDF)
Before this commit: robot COMAU_ComauSMART_NJ_500-2.7, 8 links, 7 joints
Joints:
- joint joint1: limit lower=-180 upper=180 velocity=45 -> lower=${radians(-180)} upper=${radians(180)} velocity=${radians(45)}
- joint joint2: limit lower=-60 upper=75 velocity=45 -> lower=${radians(-60)} upper=${radians(75)} velocity=${radians(45)}
- joint joint3: limit lower=-231 upper=-10 velocity=45 -> lower=${radians(-231)} upper=${radians(-10)} velocity=${radians(45)}; origin xyz=0 0 1.05 rpy=0 -90 0 -> xyz=0 0 1.05 rpy=0 ${radians(-90)} 0
- joint joint4: limit lower=-2700 upper=2700 velocity=90 -> lower=${radians(-2700)} upper=${radians(2700)} velocity=${radians(90)}
- joint joint5: limit lower=-125 upper=125 velocity=83 -> lower=${radians(-125)} upper=${radians(125)} velocity=${radians(83)}
- joint joint6: limit lower=-2700 upper=2700 velocity=130 -> lower=${radians(-2700)} upper=${radians(2700)} velocity=${radians(130)}
- joint joint_6_t-tool0: origin xyz=0.282 0 0 rpy=0 90 0 -> xyz=0.282 0 0 rpy=0 ${radians(90)} 0

File: Robots/CUSTOM_Gantry/CUSTOM_Gantry.urdf (robot description, URDF)
Before this commit: robot CUSTOM_Gantry, 8 links, 7 joints
Joints:
- joint joint4: limit lower=-30 upper=30 velocity=30 -> lower=${radians(-30)} upper=${radians(30)} velocity=${radians(30)}
- joint joint5: limit lower=-95 upper=95 velocity=30 -> lower=${radians(-95)} upper=${radians(95)} velocity=${radians(30)}
- joint joint6: limit lower=-350 upper=350 velocity=90 -> lower=${radians(-350)} upper=${radians(350)} velocity=${radians(90)}
- joint joint_6_t-tool0: origin xyz=0 0 -0.395 rpy=180 0 0 -> xyz=0 0 -0.395 rpy=${radians(180)} 0 0

File: Robots/CUSTOM_TapePlacementGantry/CUSTOM_TapePlacementGantry.urdf (robot description, URDF)
Before this commit: robot CUSTOM_TapePlacementGantry, 6 links, 5 joints
Joints:
- joint joint4: limit lower=-360 upper=360 velocity=180 -> lower=${radians(-360)} upper=${radians(360)} velocity=${radians(180)}
