Commit message: refactor UR names

File: Robots/UR10/UR10.urdf (robot description, URDF)
Before this commit: robot UR_UR5, 11 links, 10 joints
Links:
- link forearm_link: mass 2.33 -> 4.27
- link shoulder_link: mass 3.7 -> 7.1
- link upper_arm_link: mass 8.393 -> 12.7
- link wrist_1_link: mass 1.219 -> 2.0
- link wrist_2_link: mass 1.219 -> 2.0
- link wrist_3_link: mass 0.1879 -> 0.365
Joints:
- joint elbow_joint: origin xyz=-0.425 0 0 rpy=0 0 0 -> xyz=-0.612 0 0 rpy=0 0 0
- joint shoulder_lift_joint: limit lower=-6.283185307179586 upper=6.283185307179586 effort=150.0 velocity=3.141592653589793 -> lower=-6.283185307179586 upper=6.283185307179586 effort=330.0 velocity=2.0943951023931953
- joint shoulder_pan_joint: limit lower=-6.283185307179586 upper=6.283185307179586 effort=150.0 velocity=3.141592653589793 -> lower=-6.283185307179586 upper=6.283185307179586 effort=330.0 velocity=2.0943951023931953; origin xyz=0 0 0.089159 rpy=0 0 0 -> xyz=0 0 0.1273 rpy=0 0 0
- joint wrist_1_joint: limit lower=-6.283185307179586 upper=6.283185307179586 effort=28.0 velocity=3.141592653589793 -> lower=-6.283185307179586 upper=6.283185307179586 effort=56.0 velocity=3.141592653589793; origin xyz=-0.39225 0 0.10915 rpy=0 0 0 -> xyz=-0.5723 0 0.163941 rpy=0 0 0
- joint wrist_2_joint: limit lower=-6.283185307179586 upper=6.283185307179586 effort=28.0 velocity=3.141592653589793 -> lower=-6.283185307179586 upper=6.283185307179586 effort=56.0 velocity=3.141592653589793; origin xyz=0 -0.09465 -1.941303950897609e-11 rpy=1.570796327 0 0 -> xyz=0 -0.1157 -2.373046667922381e-11 rpy=1.570796327 0 0
- joint wrist_3_joint: limit lower=-6.283185307179586 upper=6.283185307179586 effort=28.0 velocity=3.141592653589793 -> lower=-6.283185307179586 upper=6.283185307179586 effort=56.0 velocity=3.141592653589793; origin xyz=0 0.0823 -1.688001216681175e-11 rpy=1.570796326589793 3.141592653589793 3.141592653589793 -> xyz=0 0.0922 -1.891053610911353e-11 rpy=1.570796326589793 3.141592653589793 3.141592653589793

File: Robots/UR10E/UR10E.urdf (robot description, URDF)
Before this commit: robot UR_UR3E, 11 links, 10 joints
Links:
- link base_link_inertia: mass 2.0 -> 4.0
- link forearm_link: mass 1.437 -> 3.989
- link shoulder_link: mass 1.98 -> 7.369
- link upper_arm_link: mass 3.4445 -> 13.051
- link wrist_1_link: mass 0.871 -> 2.1
- link wrist_2_link: mass 0.805 -> 1.98
- link wrist_3_link: mass 0.261 -> 0.615
Joints:
- joint elbow_joint: limit lower=-3.141592653589793 upper=3.141592653589793 effort=28.0 velocity=3.141592653589793 -> lower=-3.141592653589793 upper=3.141592653589793 effort=150.0 velocity=3.141592653589793; origin xyz=-0.24355 0 0 rpy=0 0 0 -> xyz=-0.6127 0 0 rpy=0 0 0
- joint shoulder_lift_joint: limit lower=-6.283185307179586 upper=6.283185307179586 effort=54.0 velocity=3.141592653589793 -> lower=-6.283185307179586 upper=6.283185307179586 effort=330.0 velocity=2.0943951023931953
- joint shoulder_pan_joint: limit lower=-6.283185307179586 upper=6.283185307179586 effort=54.0 velocity=3.141592653589793 -> lower=-6.283185307179586 upper=6.283185307179586 effort=330.0 velocity=2.0943951023931953; origin xyz=0 0 0.15185 rpy=0 0 0 -> xyz=0 0 0.1807 rpy=0 0 0
- joint wrist_1_joint: limit lower=-6.283185307179586 upper=6.283185307179586 effort=9.0 velocity=6.283185307179586 -> lower=-6.283185307179586 upper=6.283185307179586 effort=54.0 velocity=3.141592653589793; origin xyz=-0.2132 0 0.13105 rpy=0 0 0 -> xyz=-0.57155 0 0.17415 rpy=0 0 0
- joint wrist_2_joint: limit lower=-6.283185307179586 upper=6.283185307179586 effort=9.0 velocity=6.283185307179586 -> lower=-6.283185307179586 upper=6.283185307179586 effort=54.0 velocity=3.141592653589793; origin xyz=0 -0.08535 -1.750557762378351e-11 rpy=1.570796327 0 0 -> xyz=0 -0.11985 -2.458164590756244e-11 rpy=1.570796327 0 0
- joint wrist_3_joint: limit lower=-6.283185307179586 upper=6.283185307179586 effort=9.0 velocity=6.283185307179586 -> lower=-6.283185307179586 upper=6.283185307179586 effort=54.0 velocity=3.141592653589793; origin xyz=0 0.0921 -1.8890025766262e-11 rpy=1.570796326589793 3.141592653589793 3.141592653589793 -> xyz=0 0.11655 -2.390480459346185e-11 rpy=1.570796326589793 3.141592653589793 3.141592653589793

File: Robots/UR12E/UR12E.urdf (robot description, URDF)
Before this commit: robot UR_UR16E, 11 links, 10 joints
Links:
- link forearm_link: mass 4.321 -> 3.989
- link upper_arm_link: mass 10.45 -> 13.051
- link wrist_1_link: mass 2.18 -> 2.1
- link wrist_2_link: mass 2.033 -> 1.98
- link wrist_3_link: mass 0.907 -> 0.615
Joints:
- joint elbow_joint: origin xyz=-0.4784 0 0 rpy=0 0 0 -> xyz=-0.6127 0 0 rpy=0 0 0
- joint wrist_1_joint: origin xyz=-0.36 0 0.17415 rpy=0 0 0 -> xyz=-0.57155 0 0.17415 rpy=0 0 0

File: Robots/UR15/UR15.urdf (robot description, URDF)
Before this commit: robot UR_UR3, 11 links, 10 joints
Links:
- link base_link_inertia: mass 2.0 -> 4.0
- link forearm_link: mass 1.26 -> 6.1015
- link shoulder_link: mass 2.0 -> 9.9883
- link upper_arm_link: mass 3.42 -> 14.9255
- link wrist_1_link: mass 0.8 -> 2.089
- link wrist_2_link: mass 0.8 -> 2.0869
- link wrist_3_link: mass 0.35 -> 1.0666
Joints:
- joint elbow_joint: limit lower=-3.141592653589793 upper=3.141592653589793 effort=28.0 velocity=3.141592653589793 -> lower=-3.141592653589793 upper=3.141592653589793 effort=204.0 velocity=4.1887902047863905; origin xyz=-0.24365 0 0 rpy=0 0 0 -> xyz=-0.6475 0 0 rpy=0 0 0
- joint shoulder_lift_joint: limit lower=-6.283185307179586 upper=6.283185307179586 effort=56.0 velocity=3.141592653589793 -> lower=-6.283185307179586 upper=6.283185307179586 effort=433.0 velocity=3.141592653589793
- joint shoulder_pan_joint: limit lower=-6.283185307179586 upper=6.283185307179586 effort=56.0 velocity=3.141592653589793 -> lower=-6.283185307179586 upper=6.283185307179586 effort=433.0 velocity=3.141592653589793; origin xyz=0 0 0.1519 rpy=0 0 0 -> xyz=0 0 0.2186 rpy=0 0 0
- joint wrist_1_joint: limit lower=-6.283185307179586 upper=6.283185307179586 effort=12.0 velocity=6.283185307179586 -> lower=-6.283185307179586 upper=6.283185307179586 effort=70.0 velocity=5.235987755982989; origin xyz=-0.21325 0 0.11235 rpy=0 0 0 -> xyz=-0.5164 0 0.1824 rpy=0 0 0
- joint wrist_2_joint: limit lower=-6.283185307179586 upper=6.283185307179586 effort=12.0 velocity=6.283185307179586 -> lower=-6.283185307179586 upper=6.283185307179586 effort=70.0 velocity=5.235987755982989; origin xyz=0 -0.08535 -1.750557762378351e-11 rpy=1.570796327 0 0 -> xyz=0 -0.1361 -2.791457662093657e-11 rpy=1.570796327 0 0
- joint wrist_3_joint: limit lower=-6.283185307179586 upper=6.283185307179586 effort=12.0 velocity=6.283185307179586 -> lower=-6.283185307179586 upper=6.283185307179586 effort=70.0 velocity=5.235987755982989; origin xyz=0 0.0819 -1.679797079540562e-11 rpy=1.570796326589793 3.141592653589793 3.141592653589793 -> xyz=0 0.1434 -2.941183164909849e-11 rpy=1.570796326589793 3.141592653589793 3.141592653589793

File: Robots/UR16E/UR16E.urdf (robot description, URDF)
Before this commit: robot UR_UR30, 11 links, 10 joints
Links:
- link forearm_link: mass 7.156 -> 4.321
- link shoulder_link: mass 16.343 -> 7.369
- link upper_arm_link: mass 28.542 -> 10.45
- link wrist_1_link: mass 3.054 -> 2.18
- link wrist_2_link: mass 3.126 -> 2.033
- link wrist_3_link: mass 0.926 -> 0.907
Joints:
- joint elbow_joint: limit lower=-3.141592653589793 upper=3.141592653589793 effort=433.0 velocity=2.6179938779914944 -> lower=-3.141592653589793 upper=3.141592653589793 effort=150.0 velocity=3.141592653589793; origin xyz=-0.637 0 0 rpy=0 0 0 -> xyz=-0.4784 0 0 rpy=0 0 0
- joint shoulder_lift_joint: limit lower=-6.283185307179586 upper=6.283185307179586 effort=738.0 velocity=2.0943951023931953 -> lower=-6.283185307179586 upper=6.283185307179586 effort=330.0 velocity=2.0943951023931953
- joint shoulder_pan_joint: limit lower=-6.283185307179586 upper=6.283185307179586 effort=738.0 velocity=2.0943951023931953 -> lower=-6.283185307179586 upper=6.283185307179586 effort=330.0 velocity=2.0943951023931953; origin xyz=0 0 0.2363 rpy=0 0 0 -> xyz=0 0 0.1807 rpy=0 0 0
- joint wrist_1_joint: limit lower=-6.283185307179586 upper=6.283185307179586 effort=107.0 velocity=3.6651914291880923 -> lower=-6.283185307179586 upper=6.283185307179586 effort=54.0 velocity=3.141592653589793; origin xyz=-0.5037 0 0.201 rpy=0 0 0 -> xyz=-0.36 0 0.17415 rpy=0 0 0
- joint wrist_2_joint: limit lower=-6.283185307179586 upper=6.283185307179586 effort=107.0 velocity=3.6651914291880923 -> lower=-6.283185307179586 upper=6.283185307179586 effort=54.0 velocity=3.141592653589793; origin xyz=0 -0.1593 -3.267297616249225e-11 rpy=1.570796327 0 0 -> xyz=0 -0.11985 -2.458164590756244e-11 rpy=1.570796327 0 0
- joint wrist_3_joint: limit lower=-6.283185307179586 upper=6.283185307179586 effort=107.0 velocity=3.6651914291880923 -> lower=-6.283185307179586 upper=6.283185307179586 effort=54.0 velocity=3.141592653589793; origin xyz=0 0.1543 -3.16474590199156e-11 rpy=1.570796326589793 3.141592653589793 3.141592653589793 -> xyz=0 0.11655 -2.390480459346185e-11 rpy=1.570796326589793 3.141592653589793 3.141592653589793

File: Robots/UR18/UR18.urdf (robot description, URDF)
Before this commit: robot UR_UR12E, 11 links, 10 joints
Links:
- link forearm_link: mass 3.989 -> 5.52
- link shoulder_link: mass 7.369 -> 9.9883
- link upper_arm_link: mass 13.051 -> 14.2009
- link wrist_1_link: mass 2.1 -> 2.089
- link wrist_2_link: mass 1.98 -> 2.0869
- link wrist_3_link: mass 0.615 -> 1.0666
Joints:
- joint elbow_joint: limit lower=-3.141592653589793 upper=3.141592653589793 effort=150.0 velocity=3.141592653589793 -> lower=-3.141592653589793 upper=3.141592653589793 effort=204.0 velocity=4.1887902047863905; origin xyz=-0.6127 0 0 rpy=0 0 0 -> xyz=-0.475 0 0 rpy=0 0 0
- joint shoulder_lift_joint: limit lower=-6.283185307179586 upper=6.283185307179586 effort=330.0 velocity=2.0943951023931953 -> lower=-6.283185307179586 upper=6.283185307179586 effort=433.0 velocity=3.141592653589793
- joint shoulder_pan_joint: limit lower=-6.283185307179586 upper=6.283185307179586 effort=330.0 velocity=2.0943951023931953 -> lower=-6.283185307179586 upper=6.283185307179586 effort=433.0 velocity=3.141592653589793; origin xyz=0 0 0.1807 rpy=0 0 0 -> xyz=0 0 0.2186 rpy=0 0 0
- joint wrist_1_joint: limit lower=-6.283185307179586 upper=6.283185307179586 effort=54.0 velocity=3.141592653589793 -> lower=-6.283185307179586 upper=6.283185307179586 effort=70.0 velocity=5.235987755982989; origin xyz=-0.57155 0 0.17415 rpy=0 0 0 -> xyz=-0.3389 0 0.1824 rpy=0 0 0
- joint wrist_2_joint: limit lower=-6.283185307179586 upper=6.283185307179586 effort=54.0 velocity=3.141592653589793 -> lower=-6.283185307179586 upper=6.283185307179586 effort=70.0 velocity=5.235987755982989; origin xyz=0 -0.11985 -2.458164590756244e-11 rpy=1.570796327 0 0 -> xyz=0 -0.1361 -2.791457662093657e-11 rpy=1.570796327 0 0
- joint wrist_3_joint: limit lower=-6.283185307179586 upper=6.283185307179586 effort=54.0 velocity=3.141592653589793 -> lower=-6.283185307179586 upper=6.283185307179586 effort=70.0 velocity=5.235987755982989; origin xyz=0 0.11655 -2.390480459346185e-11 rpy=1.570796326589793 3.141592653589793 3.141592653589793 -> xyz=0 0.1434 -2.941183164909849e-11 rpy=1.570796326589793 3.141592653589793 3.141592653589793

File: Robots/UR20/UR20.urdf (robot description, URDF)
Before this commit: robot UR_UR15, 11 links, 10 joints
Links:
- link forearm_link: mass 6.1015 -> 7.879
- link shoulder_link: mass 9.9883 -> 16.343
- link upper_arm_link: mass 14.9255 -> 29.632
- link wrist_1_link: mass 2.089 -> 3.054
- link wrist_2_link: mass 2.0869 -> 3.126
- link wrist_3_link: mass 1.0666 -> 0.926
Joints:
- joint elbow_joint: limit lower=-3.141592653589793 upper=3.141592653589793 effort=204.0 velocity=4.1887902047863905 -> lower=-3.141592653589793 upper=3.141592653589793 effort=433.0 velocity=2.6179938779914944; origin xyz=-0.6475 0 0 rpy=0 0 0 -> xyz=-0.862 0 0 rpy=0 0 0
- joint shoulder_lift_joint: limit lower=-6.283185307179586 upper=6.283185307179586 effort=433.0 velocity=3.141592653589793 -> lower=-6.283185307179586 upper=6.283185307179586 effort=738.0 velocity=2.0943951023931953
- joint shoulder_pan_joint: limit lower=-6.283185307179586 upper=6.283185307179586 effort=433.0 velocity=3.141592653589793 -> lower=-6.283185307179586 upper=6.283185307179586 effort=738.0 velocity=2.0943951023931953; origin xyz=0 0 0.2186 rpy=0 0 0 -> xyz=0 0 0.2363 rpy=0 0 0
- joint wrist_1_joint: limit lower=-6.283185307179586 upper=6.283185307179586 effort=70.0 velocity=5.235987755982989 -> lower=-6.283185307179586 upper=6.283185307179586 effort=107.0 velocity=3.6651914291880923; origin xyz=-0.5164 0 0.1824 rpy=0 0 0 -> xyz=-0.7287 0 0.201 rpy=0 0 0
- joint wrist_2_joint: limit lower=-6.283185307179586 upper=6.283185307179586 effort=70.0 velocity=5.235987755982989 -> lower=-6.283185307179586 upper=6.283185307179586 effort=107.0 velocity=3.6651914291880923; origin xyz=0 -0.1361 -2.791457662093657e-11 rpy=1.570796327 0 0 -> xyz=0 -0.1593 -3.267297616249225e-11 rpy=1.570796327 0 0
- joint wrist_3_joint: limit lower=-6.283185307179586 upper=6.283185307179586 effort=70.0 velocity=5.235987755982989 -> lower=-6.283185307179586 upper=6.283185307179586 effort=107.0 velocity=3.6651914291880923; origin xyz=0 0.1434 -2.941183164909849e-11 rpy=1.570796326589793 3.141592653589793 3.141592653589793 -> xyz=0 0.1543 -3.1647459019915597e-11 rpy=1.570796326589793 3.141592653589793 3.141592653589793

File: Robots/UR3/UR3.urdf (robot description, URDF)
Before this commit: robot UR_UR7E, 11 links, 10 joints
Links:
- link base_link_inertia: mass 4.0 -> 2.0
- link forearm_link: mass 2.846 -> 1.26
- link shoulder_link: mass 3.761 -> 2.0
- link upper_arm_link: mass 8.058 -> 3.42
- link wrist_1_link: mass 1.37 -> 0.8
- link wrist_2_link: mass 1.3 -> 0.8
- link wrist_3_link: mass 0.365 -> 0.35
Joints:
- joint elbow_joint: limit lower=-3.141592653589793 upper=3.141592653589793 effort=150.0 velocity=3.141592653589793 -> lower=-3.141592653589793 upper=3.141592653589793 effort=28.0 velocity=3.141592653589793; origin xyz=-0.425 0 0 rpy=0 0 0 -> xyz=-0.24365 0 0 rpy=0 0 0
- joint shoulder_lift_joint: limit lower=-6.283185307179586 upper=6.283185307179586 effort=150.0 velocity=3.141592653589793 -> lower=-6.283185307179586 upper=6.283185307179586 effort=56.0 velocity=3.141592653589793
- joint shoulder_pan_joint: limit lower=-6.283185307179586 upper=6.283185307179586 effort=150.0 velocity=3.141592653589793 -> lower=-6.283185307179586 upper=6.283185307179586 effort=56.0 velocity=3.141592653589793; origin xyz=0 0 0.1625 rpy=0 0 0 -> xyz=0 0 0.1519 rpy=0 0 0
- joint wrist_1_joint: limit lower=-6.283185307179586 upper=6.283185307179586 effort=28.0 velocity=3.141592653589793 -> lower=-6.283185307179586 upper=6.283185307179586 effort=12.0 velocity=6.283185307179586; origin xyz=-0.3922 0 0.1333 rpy=0 0 0 -> xyz=-0.21325 0 0.11235 rpy=0 0 0
- joint wrist_2_joint: limit lower=-6.283185307179586 upper=6.283185307179586 effort=28.0 velocity=3.141592653589793 -> lower=-6.283185307179586 upper=6.283185307179586 effort=12.0 velocity=6.283185307179586; origin xyz=0 -0.0997 -2.044881182297852e-11 rpy=1.570796327 0 0 -> xyz=0 -0.08535 -1.750557762378351e-11 rpy=1.570796327 0 0
- joint wrist_3_joint: limit lower=-6.283185307179586 upper=6.283185307179586 effort=28.0 velocity=3.141592653589793 -> lower=-6.283185307179586 upper=6.283185307179586 effort=12.0 velocity=6.283185307179586; origin xyz=0 0.0996 -2.042830148012698e-11 rpy=1.570796326589793 3.141592653589793 3.141592653589793 -> xyz=0 0.0819 -1.679797079540562e-11 rpy=1.570796326589793 3.141592653589793 3.141592653589793

File: Robots/UR30/UR30.urdf (robot description, URDF)
Before this commit: robot UR_UR18, 11 links, 10 joints
Links:
- link forearm_link: mass 5.52 -> 7.156
- link shoulder_link: mass 9.9883 -> 16.343
- link upper_arm_link: mass 14.2009 -> 28.542
- link wrist_1_link: mass 2.089 -> 3.054
- link wrist_2_link: mass 2.0869 -> 3.126
- link wrist_3_link: mass 1.0666 -> 0.926
Joints:
- joint elbow_joint: limit lower=-3.141592653589793 upper=3.141592653589793 effort=204.0 velocity=4.1887902047863905 -> lower=-3.141592653589793 upper=3.141592653589793 effort=433.0 velocity=2.6179938779914944; origin xyz=-0.475 0 0 rpy=0 0 0 -> xyz=-0.637 0 0 rpy=0 0 0
- joint shoulder_lift_joint: limit lower=-6.283185307179586 upper=6.283185307179586 effort=433.0 velocity=3.141592653589793 -> lower=-6.283185307179586 upper=6.283185307179586 effort=738.0 velocity=2.0943951023931953
- joint shoulder_pan_joint: limit lower=-6.283185307179586 upper=6.283185307179586 effort=433.0 velocity=3.141592653589793 -> lower=-6.283185307179586 upper=6.283185307179586 effort=738.0 velocity=2.0943951023931953; origin xyz=0 0 0.2186 rpy=0 0 0 -> xyz=0 0 0.2363 rpy=0 0 0
- joint wrist_1_joint: limit lower=-6.283185307179586 upper=6.283185307179586 effort=70.0 velocity=5.235987755982989 -> lower=-6.283185307179586 upper=6.283185307179586 effort=107.0 velocity=3.6651914291880923; origin xyz=-0.3389 0 0.1824 rpy=0 0 0 -> xyz=-0.5037 0 0.201 rpy=0 0 0
- joint wrist_2_joint: limit lower=-6.283185307179586 upper=6.283185307179586 effort=70.0 velocity=5.235987755982989 -> lower=-6.283185307179586 upper=6.283185307179586 effort=107.0 velocity=3.6651914291880923; origin xyz=0 -0.1361 -2.791457662093657e-11 rpy=1.570796327 0 0 -> xyz=0 -0.1593 -3.267297616249225e-11 rpy=1.570796327 0 0
- joint wrist_3_joint: limit lower=-6.283185307179586 upper=6.283185307179586 effort=70.0 velocity=5.235987755982989 -> lower=-6.283185307179586 upper=6.283185307179586 effort=107.0 velocity=3.6651914291880923; origin xyz=0 0.1434 -2.941183164909849e-11 rpy=1.570796326589793 3.141592653589793 3.141592653589793 -> xyz=0 0.1543 -3.16474590199156e-11 rpy=1.570796326589793 3.141592653589793 3.141592653589793

File: Robots/UR3E/UR3E.urdf (robot description, URDF)
Before this commit: robot UR_UR8LONG, 11 links, 10 joints
Links:
- link base_link_inertia: mass 4.0 -> 2.0
- link forearm_link: mass 7.6393 -> 1.437
- link shoulder_link: mass 9.9883 -> 1.98
- link upper_arm_link: mass 17.0738 -> 3.4445
- link wrist_1_link: mass 2.089 -> 0.871
- link wrist_2_link: mass 2.0869 -> 0.805
- link wrist_3_link: mass 1.0666 -> 0.261
Joints:
- joint elbow_joint: limit lower=-3.141592653589793 upper=3.141592653589793 effort=204.0 velocity=4.1887902047863905 -> lower=-3.141592653589793 upper=3.141592653589793 effort=28.0 velocity=3.141592653589793; origin xyz=-0.8989 0 0 rpy=0 0 0 -> xyz=-0.24355 0 0 rpy=0 0 0
- joint shoulder_lift_joint: limit lower=-6.283185307179586 upper=6.283185307179586 effort=433.0 velocity=3.141592653589793 -> lower=-6.283185307179586 upper=6.283185307179586 effort=54.0 velocity=3.141592653589793
- joint shoulder_pan_joint: limit lower=-6.283185307179586 upper=6.283185307179586 effort=433.0 velocity=3.141592653589793 -> lower=-6.283185307179586 upper=6.283185307179586 effort=54.0 velocity=3.141592653589793; origin xyz=0 0 0.2186 rpy=0 0 0 -> xyz=0 0 0.15185 rpy=0 0 0
- joint wrist_1_joint: limit lower=-6.283185307179586 upper=6.283185307179586 effort=70.0 velocity=5.235987755982989 -> lower=-6.283185307179586 upper=6.283185307179586 effort=9.0 velocity=6.283185307179586; origin xyz=-0.7149 0 0.1824 rpy=0 0 0 -> xyz=-0.2132 0 0.13105 rpy=0 0 0
- joint wrist_2_joint: limit lower=-6.283185307179586 upper=6.283185307179586 effort=70.0 velocity=5.235987755982989 -> lower=-6.283185307179586 upper=6.283185307179586 effort=9.0 velocity=6.283185307179586; origin xyz=0 -0.1361 -2.791457662093657e-11 rpy=1.570796327 0 0 -> xyz=0 -0.08535 -1.750557762378351e-11 rpy=1.570796327 0 0
- joint wrist_3_joint: limit lower=-6.283185307179586 upper=6.283185307179586 effort=70.0 velocity=5.235987755982989 -> lower=-6.283185307179586 upper=6.283185307179586 effort=9.0 velocity=6.283185307179586; origin xyz=0 0.1434 -2.941183164909849e-11 rpy=1.570796326589793 3.141592653589793 3.141592653589793 -> xyz=0 0.0921 -1.8890025766262e-11 rpy=1.570796326589793 3.141592653589793 3.141592653589793

File: Robots/UR5/UR5.urdf (robot description, URDF)
Before this commit: robot UR_UR10, 11 links, 10 joints
Links:
- link forearm_link: mass 4.27 -> 2.33
- link shoulder_link: mass 7.1 -> 3.7
- link upper_arm_link: mass 12.7 -> 8.393
- link wrist_1_link: mass 2.0 -> 1.219
- link wrist_2_link: mass 2.0 -> 1.219
- link wrist_3_link: mass 0.365 -> 0.1879
Joints:
- joint elbow_joint: origin xyz=-0.612 0 0 rpy=0 0 0 -> xyz=-0.425 0 0 rpy=0 0 0
- joint shoulder_lift_joint: limit lower=-6.283185307179586 upper=6.283185307179586 effort=330.0 velocity=2.0943951023931953 -> lower=-6.283185307179586 upper=6.283185307179586 effort=150.0 velocity=3.141592653589793
- joint shoulder_pan_joint: limit lower=-6.283185307179586 upper=6.283185307179586 effort=330.0 velocity=2.0943951023931953 -> lower=-6.283185307179586 upper=6.283185307179586 effort=150.0 velocity=3.141592653589793; origin xyz=0 0 0.1273 rpy=0 0 0 -> xyz=0 0 0.089159 rpy=0 0 0
- joint wrist_1_joint: limit lower=-6.283185307179586 upper=6.283185307179586 effort=56.0 velocity=3.141592653589793 -> lower=-6.283185307179586 upper=6.283185307179586 effort=28.0 velocity=3.141592653589793; origin xyz=-0.5723 0 0.163941 rpy=0 0 0 -> xyz=-0.39225 0 0.10915 rpy=0 0 0
- joint wrist_2_joint: limit lower=-6.283185307179586 upper=6.283185307179586 effort=56.0 velocity=3.141592653589793 -> lower=-6.283185307179586 upper=6.283185307179586 effort=28.0 velocity=3.141592653589793; origin xyz=0 -0.1157 -2.373046667922381e-11 rpy=1.570796327 0 0 -> xyz=0 -0.09465 -1.941303950897609e-11 rpy=1.570796327 0 0
- joint wrist_3_joint: limit lower=-6.283185307179586 upper=6.283185307179586 effort=56.0 velocity=3.141592653589793 -> lower=-6.283185307179586 upper=6.283185307179586 effort=28.0 velocity=3.141592653589793; origin xyz=0 0.0922 -1.891053610911353e-11 rpy=1.570796326589793 3.141592653589793 3.141592653589793 -> xyz=0 0.0823 -1.688001216681175e-11 rpy=1.570796326589793 3.141592653589793 3.141592653589793
