Commit message: refactor UR names

File: Robots/UR5E/UR5E.urdf (robot description, URDF)
Before this commit: robot UR_UR20, 11 links, 10 joints
Links:
- link forearm_link: mass 7.879 -> 2.846
- link shoulder_link: mass 16.343 -> 3.761
- link upper_arm_link: mass 29.632 -> 8.058
- link wrist_1_link: mass 3.054 -> 1.37
- link wrist_2_link: mass 3.126 -> 1.3
- link wrist_3_link: mass 0.926 -> 0.365
Joints:
- joint elbow_joint: limit lower=-3.141592653589793 upper=3.141592653589793 effort=433.0 velocity=2.6179938779914944 -> lower=-3.141592653589793 upper=3.141592653589793 effort=150.0 velocity=3.141592653589793; origin xyz=-0.862 0 0 rpy=0 0 0 -> xyz=-0.425 0 0 rpy=0 0 0
- joint shoulder_lift_joint: limit lower=-6.283185307179586 upper=6.283185307179586 effort=738.0 velocity=2.0943951023931953 -> lower=-6.283185307179586 upper=6.283185307179586 effort=150.0 velocity=3.141592653589793
- joint shoulder_pan_joint: limit lower=-6.283185307179586 upper=6.283185307179586 effort=738.0 velocity=2.0943951023931953 -> lower=-6.283185307179586 upper=6.283185307179586 effort=150.0 velocity=3.141592653589793; origin xyz=0 0 0.2363 rpy=0 0 0 -> xyz=0 0 0.1625 rpy=0 0 0
- joint wrist_1_joint: limit lower=-6.283185307179586 upper=6.283185307179586 effort=107.0 velocity=3.6651914291880923 -> lower=-6.283185307179586 upper=6.283185307179586 effort=28.0 velocity=3.141592653589793; origin xyz=-0.7287 0 0.201 rpy=0 0 0 -> xyz=-0.3922 0 0.1333 rpy=0 0 0
- joint wrist_2_joint: limit lower=-6.283185307179586 upper=6.283185307179586 effort=107.0 velocity=3.6651914291880923 -> lower=-6.283185307179586 upper=6.283185307179586 effort=28.0 velocity=3.141592653589793; origin xyz=0 -0.1593 -3.267297616249225e-11 rpy=1.570796327 0 0 -> xyz=0 -0.0997 -2.044881182297852e-11 rpy=1.570796327 0 0
- joint wrist_3_joint: limit lower=-6.283185307179586 upper=6.283185307179586 effort=107.0 velocity=3.6651914291880923 -> lower=-6.283185307179586 upper=6.283185307179586 effort=28.0 velocity=3.141592653589793; origin xyz=0 0.1543 -3.1647459019915597e-11 rpy=1.570796326589793 3.141592653589793 3.141592653589793 -> xyz=0 0.0996 -2.042830148012698e-11 rpy=1.570796326589793 3.141592653589793 3.141592653589793

File: Robots/UR8LONG/UR8LONG.urdf (robot description, URDF)
Before this commit: robot UR_UR10E, 11 links, 10 joints
Links:
- link forearm_link: mass 3.989 -> 7.6393
- link shoulder_link: mass 7.369 -> 9.9883
- link upper_arm_link: mass 13.051 -> 17.0738
- link wrist_1_link: mass 2.1 -> 2.089
- link wrist_2_link: mass 1.98 -> 2.0869
- link wrist_3_link: mass 0.615 -> 1.0666
Joints:
- joint elbow_joint: limit lower=-3.141592653589793 upper=3.141592653589793 effort=150.0 velocity=3.141592653589793 -> lower=-3.141592653589793 upper=3.141592653589793 effort=204.0 velocity=4.1887902047863905; origin xyz=-0.6127 0 0 rpy=0 0 0 -> xyz=-0.8989 0 0 rpy=0 0 0
- joint shoulder_lift_joint: limit lower=-6.283185307179586 upper=6.283185307179586 effort=330.0 velocity=2.0943951023931953 -> lower=-6.283185307179586 upper=6.283185307179586 effort=433.0 velocity=3.141592653589793
- joint shoulder_pan_joint: limit lower=-6.283185307179586 upper=6.283185307179586 effort=330.0 velocity=2.0943951023931953 -> lower=-6.283185307179586 upper=6.283185307179586 effort=433.0 velocity=3.141592653589793; origin xyz=0 0 0.1807 rpy=0 0 0 -> xyz=0 0 0.2186 rpy=0 0 0
- joint wrist_1_joint: limit lower=-6.283185307179586 upper=6.283185307179586 effort=54.0 velocity=3.141592653589793 -> lower=-6.283185307179586 upper=6.283185307179586 effort=70.0 velocity=5.235987755982989; origin xyz=-0.57155 0 0.17415 rpy=0 0 0 -> xyz=-0.7149 0 0.1824 rpy=0 0 0
- joint wrist_2_joint: limit lower=-6.283185307179586 upper=6.283185307179586 effort=54.0 velocity=3.141592653589793 -> lower=-6.283185307179586 upper=6.283185307179586 effort=70.0 velocity=5.235987755982989; origin xyz=0 -0.11985 -2.458164590756244e-11 rpy=1.570796327 0 0 -> xyz=0 -0.1361 -2.791457662093657e-11 rpy=1.570796327 0 0
- joint wrist_3_joint: limit lower=-6.283185307179586 upper=6.283185307179586 effort=54.0 velocity=3.141592653589793 -> lower=-6.283185307179586 upper=6.283185307179586 effort=70.0 velocity=5.235987755982989; origin xyz=0 0.11655 -2.390480459346185e-11 rpy=1.570796326589793 3.141592653589793 3.141592653589793 -> xyz=0 0.1434 -2.941183164909849e-11 rpy=1.570796326589793 3.141592653589793 3.141592653589793
