Commit message: change joint angle units

File: Robots/INOVANCE_IR-R35JQR/INOVANCE_IR-R35JQR.urdf (robot description, URDF)
Before this commit: robot INOVANCE_IR-R35JQR, 8 links, 7 joints
Joints:
- joint joint1: limit lower=-170 upper=170 velocity=200 -> lower=${radians(-170)} upper=${radians(170)} velocity=${radians(200)}
- joint joint2: limit lower=-155 upper=80 velocity=180 -> lower=${radians(-155)} upper=${radians(80)} velocity=${radians(180)}
- joint joint3: limit lower=-160 upper=75 velocity=242 -> lower=${radians(-160)} upper=${radians(75)} velocity=${radians(242)}
- joint joint4: limit lower=-180 upper=180 velocity=450 -> lower=${radians(-180)} upper=${radians(180)} velocity=${radians(450)}
- joint joint5: limit lower=-130 upper=130 velocity=336 -> lower=${radians(-130)} upper=${radians(130)} velocity=${radians(336)}
- joint joint6: limit lower=-360 upper=360 velocity=407 -> lower=${radians(-360)} upper=${radians(360)} velocity=${radians(407)}
- joint joint_6_t-tool0: origin xyz=0.13 0 0 rpy=0 90 0 -> xyz=0.13 0 0 rpy=0 ${radians(90)} 0

File: Robots/KUKA_KR10R1420HP/KUKA_KR10R1420HP.urdf (robot description, URDF)
Before this commit: robot KUKA_KR10R1420HP, 8 links, 7 joints
Joints:
- joint joint1: limit lower=-170 upper=170 velocity=220 -> lower=${radians(-170)} upper=${radians(170)} velocity=${radians(220)}
- joint joint2: limit lower=-185 upper=65 velocity=210 -> lower=${radians(-185)} upper=${radians(65)} velocity=${radians(210)}
- joint joint3: limit lower=-137 upper=163 velocity=270 -> lower=${radians(-137)} upper=${radians(163)} velocity=${radians(270)}
- joint joint4: limit lower=-185 upper=185 velocity=381 -> lower=${radians(-185)} upper=${radians(185)} velocity=${radians(381)}
- joint joint5: limit lower=-120 upper=120 velocity=311 -> lower=${radians(-120)} upper=${radians(120)} velocity=${radians(311)}
- joint joint6: limit lower=-350 upper=350 velocity=492 -> lower=${radians(-350)} upper=${radians(350)} velocity=${radians(492)}
- joint joint_6_t-tool0: origin xyz=0 0 0 rpy=0 90 0 -> xyz=0 0 0 rpy=0 ${radians(90)} 0

File: Robots/KUKA_KR210R2700-2/KUKA_KR210R2700-2.urdf (robot description, URDF)
Before this commit: robot KUKA_KR210R2700-2, 8 links, 7 joints
Joints:
- joint joint1: limit lower=-185 upper=185 velocity=120 -> lower=${radians(-185)} upper=${radians(185)} velocity=${radians(120)}
- joint joint2: limit lower=-140 upper=-5 velocity=115 -> lower=${radians(-140)} upper=${radians(-5)} velocity=${radians(115)}; origin xyz=0.33 0 0 rpy=0 90 0 -> xyz=0.33 0 0 rpy=0 ${radians(90)} 0
- joint joint3: limit lower=-120 upper=168 velocity=112 -> lower=${radians(-120)} upper=${radians(168)} velocity=${radians(112)}; origin xyz=0 0 1.15 rpy=0 -90 0 -> xyz=0 0 1.15 rpy=0 ${radians(-90)} 0
- joint joint4: limit lower=-350 upper=350 velocity=179 -> lower=${radians(-350)} upper=${radians(350)} velocity=${radians(179)}
- joint joint5: limit lower=-125 upper=150 velocity=172 -> lower=${radians(-125)} upper=${radians(150)} velocity=${radians(172)}
- joint joint6: limit lower=-350 upper=350 velocity=220 -> lower=${radians(-350)} upper=${radians(350)} velocity=${radians(220)}
- joint joint_6_t-tool0: origin xyz=0.215 0 0 rpy=0 90 0 -> xyz=0.215 0 0 rpy=0 ${radians(90)} 0

File: Robots/KUKA_KR360R2830/KUKA_KR360R2830.urdf (robot description, URDF)
Before this commit: robot KUKA_KR360R2830, 8 links, 7 joints
Joints:
- joint joint1: limit lower=-185 upper=185 velocity=100 -> lower=${radians(-185)} upper=${radians(185)} velocity=${radians(100)}
- joint joint2: limit lower=-130 upper=20 velocity=90 -> lower=${radians(-130)} upper=${radians(20)} velocity=${radians(90)}; origin xyz=0.5 0 1.045 rpy=0 90 0 -> xyz=0.5 0 1.045 rpy=0 ${radians(90)} 0
- joint joint3: limit lower=-100 upper=144 velocity=90 -> lower=${radians(-100)} upper=${radians(144)} velocity=${radians(90)}; origin xyz=0 0 1.3 rpy=0 -90 0 -> xyz=0 0 1.3 rpy=0 ${radians(-90)} 0
- joint joint4: limit lower=-350 upper=350 velocity=120 -> lower=${radians(-350)} upper=${radians(350)} velocity=${radians(120)}
- joint joint5: limit lower=-120 upper=120 velocity=110 -> lower=${radians(-120)} upper=${radians(120)} velocity=${radians(110)}
- joint joint6: limit lower=-350 upper=350 velocity=160 -> lower=${radians(-350)} upper=${radians(350)} velocity=${radians(160)}
- joint joint_6_t-tool0: origin xyz=0.29 0 0 rpy=0 90 0 -> xyz=0.29 0 0 rpy=0 ${radians(90)} 0

File: Robots/KUKA_KR480R3330MT/KUKA_KR480R3330MT.urdf (robot description, URDF)
Before this commit: robot KUKA_KR480R3330MT, 8 links, 7 joints
Joints:
- joint joint1: limit lower=-185 upper=185 velocity=45 -> lower=${radians(-185)} upper=${radians(185)} velocity=${radians(45)}
- joint joint2: limit lower=-130 upper=20 velocity=45 -> lower=${radians(-130)} upper=${radians(20)} velocity=${radians(45)}; origin xyz=0.5 0 1.045 rpy=0 90 0 -> xyz=0.5 0 1.045 rpy=0 ${radians(90)} 0
- joint joint3: limit lower=-100 upper=144 velocity=45 -> lower=${radians(-100)} upper=${radians(144)} velocity=${radians(45)}; origin xyz=0 0 1.3 rpy=0 -90 0 -> xyz=0 0 1.3 rpy=0 ${radians(-90)} 0
- joint joint4: limit lower=-350 upper=350 velocity=90 -> lower=${radians(-350)} upper=${radians(350)} velocity=${radians(90)}
- joint joint5: limit lower=-120 upper=120 velocity=83 -> lower=${radians(-120)} upper=${radians(120)} velocity=${radians(83)}
- joint joint6: limit lower=-350 upper=350 velocity=130 -> lower=${radians(-350)} upper=${radians(350)} velocity=${radians(130)}
- joint joint_6_t-tool0: origin xyz=0.29 0 0 rpy=0 90 0 -> xyz=0.29 0 0 rpy=0 ${radians(90)} 0

File: Robots/KUKA_KR500R2380/KUKA_KR500R2380.urdf (robot description, URDF)
Before this commit: robot KUKA_KR500R2380, 8 links, 7 joints
Joints:
- joint joint1: limit lower=-185 upper=185 velocity=90 -> lower=${radians(-185)} upper=${radians(185)} velocity=${radians(90)}
- joint joint2: limit lower=-130 upper=20 velocity=80 -> lower=${radians(-130)} upper=${radians(20)} velocity=${radians(80)}; origin xyz=0.5 0 1.045 rpy=0 90 0 -> xyz=0.5 0 1.045 rpy=0 ${radians(90)} 0
- joint joint3: limit lower=-100 upper=144 velocity=75 -> lower=${radians(-100)} upper=${radians(144)} velocity=${radians(75)}; origin xyz=0 0 1.3 rpy=0 -90 0 -> xyz=0 0 1.3 rpy=0 ${radians(-90)} 0
- joint joint4: limit lower=-350 upper=350 velocity=90 -> lower=${radians(-350)} upper=${radians(350)} velocity=${radians(90)}
- joint joint5: limit lower=-120 upper=120 velocity=83 -> lower=${radians(-120)} upper=${radians(120)} velocity=${radians(83)}
- joint joint6: limit lower=-350 upper=350 velocity=130 -> lower=${radians(-350)} upper=${radians(350)} velocity=${radians(130)}
- joint joint_6_t-tool0: origin xyz=0.29 0 0 rpy=0 90 0 -> xyz=0.29 0 0 rpy=0 ${radians(90)} 0
