Commit message: fix custom gantry

File: Robots/CUSTOM_Gantry/CUSTOM_Gantry.urdf (robot description, URDF)
Before this commit: robot CUSTOM_Gantry, 8 links, 7 joints
Links:
- removed link link_1
- added link link1; collision mesh filename=collision/link_1.stl; visual mesh filename=visual/link_1.stl
Joints:
- joint joint1: child link_1 -> link1
